File: Esquema/esquemaProyecto.sch (EAGLE design)
At the start: 3 parts, among them IC1 ATMEGA644-10PU

Commit message: Esquematico y reporte
Parts:
- removed IC1: ATMEGA644-10PU, atmel:ATMEGA644-10PU
- added IC2: LP2950CZ-3.0, v-reg:LP2950CZ-3.0
- added U$3: ARDUINO-BPLACE, adafruit:ARDUINO-BPLACE
- added X1: HD44780LCD-1602, adafruit:HD44780LCD-1602
Connections:
- new net N$1: U$3.D12, X1.RS
- new net N$10: U$2.AO, U$3.A1
- new net N$11: U$2.GND, U$3.GND2
- new net N$2: U$3.D7, X1.E
- new net N$3: U$3.D11, X1.DB4
- new net N$4: U$3.D10, X1.DB5
- new net N$5: U$3.D9, X1.DB6
- new net N$6: U$3.D8, X1.DB7
- new net N$7: U$1.TRIG, U$3.D6
- new net N$8: U$1.ECHO, U$3.D5
- new net N$9: IC2.OUT, U$3.A0
- new net VDD: IC2.GND, U$1.GND, U$3.GND1, X1.A, X1.RW, X1.VDD
- new net VSS: IC2.IN, U$1.VCC, U$2.VCC, U$3.5V, X1.VSS
Changed lines of the file:
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@@
 <part name="U$1" library="diy-modules" deviceset="ULTRASONIC-HC-SR04" device=""/>
 <part name="U$2" library="diy-modules" deviceset="GAS-SENSOR-MQ2" device=""/>
-<part name="IC1" library="atmel" library_urn="urn:adsk.eagle:library:105" deviceset="ATMEGA644-*PU" device="" package3d_urn="urn:adsk.eagle:package:4314/1" technology="10"/>
+<part name="IC2" library="v-reg" library_urn="urn:adsk.eagle:library:409" deviceset="LP2950?*" device="CZ" package3d_urn="urn:adsk.eagle:package:20831/2" technology="-3.0"/>
+<part name="U$3" library="adafruit" deviceset="ARDUINO" device="-BPLACE"/>
+<part name="X1" library="adafruit" deviceset="HD44780LCD" device="-1602"/>
 </parts>
 <sheets>
@@
 <attribute name="VALUE" x="198.12" y="104.14" size="1.778" layer="96"/>
 </instance>
-<instance part="IC1" gate="G$1" x="152.4" y="139.7" smashed="yes">
-<attribute name="NAME" x="124.46" y="166.37" size="1.778" layer="95"/>
-<attribute name="VALUE" x="124.46" y="109.22" size="1.778" layer="96"/>
+<instance part="IC2" gate="G$1" x="200.66" y="187.96" smashed="yes">
+<attribute name="NAME" x="203.2" y="180.34" size="1.778" layer="95"/>
+<attribute name="VALUE" x="203.2" y="177.8" size="1.778" layer="96"/>
+</instance>
+<instance part="U$3" gate="G$1" x="144.78" y="154.94" smashed="yes"/>
+<instance part="X1" gate="G$1" x="83.82" y="185.42" smashed="yes">
+<attribute name="NAME" x="58.42" y="172.72" size="2.1844" layer="95" font="vector"/>
+<attribute name="VALUE" x="73.66" y="172.72" size="2.1844" layer="96" font="vector"/>
 </instance>
 </instances>
@@
 </busses>
 <nets>
+<net name="N$1" class="0">
+<segment>
+<pinref part="U$3" gate="G$1" pin="D12"/>
+<wire x1="142.24" y1="182.88" x2="142.24" y2="208.28" width="0.1524" layer="91"/>
+<wire x1="142.24" y1="208.28" x2="68.58" y2="208.28" width="0.1524" layer="91"/>
+<pinref part="X1" gate="G$1" pin="RS"/>
+<wire x1="68.58" y1="208.28" x2="68.58" y2="203.2" width="0.1524" layer="91"/>
+</segment>
+</net>
+<net name="N$2" class="0">
+<segment>
+<pinref part="X1" gate="G$1" pin="E"/>
+<wire x1="73.66" y1="203.2" x2="73.66" y2="218.44" width="0.1524" layer="91"/>
+<pinref part="U$3" gate="G$1" pin="D7"/>
+<wire x1="73.66" y1="218.44" x2="157.48" y2="218.44" width="0.1524" layer="91"/>
+<wire x1="157.48" y1="218.44" x2="157.48" y2="182.88" width="0.1524" layer="91"/>
+</segment>
+</net>
+<net name="N$3" class="0">
+<segment>
+<pinref part="X1" gate="G$1" pin="DB4"/>
+<wire x1="86.36" y1="203.2" x2="86.36" y2="215.9" width="0.1524" layer="91"/>
+<pinref part="U$3" gate="G$1" pin="D11"/>
+<wire x1="86.36" y1="215.9" x2="144.78" y2="215.9" width="0.1524" layer="91"/>
+<wire x1="144.78" y1="215.9" x2="144.78" y2="182.88" width="0.1524" layer="91"/>
+</segment>
+</net>
+<net name="N$4" class="0">
+<segment>
+<pinref part="X1" gate="G$1" pin="DB5"/>
+<wire x1="88.9" y1="203.2" x2="88.9" y2="213.36" width="0.1524" layer="91"/>
+<wire x1="88.9" y1="213.36" x2="147.32" y2="213.36" width="0.1524" layer="91"/>
+<pinref part="U$3" gate="G$1" pin="D10"/>
+<wire x1="147.32" y1="213.36" x2="147.32" y2="182.88" width="0.1524" layer="91"/>
+</segment>
+</net>
+<net name="N$5" class="0">
+<segment>
+<pinref part="X1" gate="G$1" pin="DB6"/>
+<wire x1="91.44" y1="203.2" x2="91.44" y2="210.82" width="0.1524" layer="91"/>
+<pinref part="U$3" gate="G$1" pin="D9"/>
+<wire x1="91.44" y1="210.82" x2="149.86" y2="210.82" width="0.1524" layer="91"/>
+<wire x1="149.86" y1="210.82" x2="149.86" y2="182.88" width="0.1524" layer="91"/>
+</segment>
+</net>
+<net name="N$6" class="0">
+<segment>
+<pinref part="X1" gate="G$1" pin="DB7"/>
+<wire x1="93.98" y1="203.2" x2="93.98" y2="223.52" width="0.1524" layer="91"/>
+<pinref part="U$3" gate="G$1" pin="D8"/>
+<wire x1="93.98" y1="223.52" x2="152.4" y2="223.52" width="0.1524" layer="91"/>
+<wire x1="152.4" y1="223.52" x2="152.4" y2="182.88" width="0.1524" layer="91"/>
+</segment>
+</net>
+<net name="N$7" class="0">
+<segment>
+<pinref part="U$3" gate="G$1" pin="D6"/>
+<wire x1="160.02" y1="182.88" x2="160.02" y2="142.24" width="0.1524" layer="91"/>
+<wire x1="160.02" y1="142.24" x2="114.3" y2="142.24" width="0.1524" layer="91"/>
+<wire x1="114.3" y1="142.24" x2="114.3" y2="116.84" width="0.1524" layer="91"/>
+<wire x1="114.3" y1="116.84" x2="81.28" y2="116.84" width="0.1524" layer="91"/>
+<pinref part="U$1" gate="G$1" pin="TRIG"/>
+<wire x1="81.28" y1="116.84" x2="81.28" y2="134.62" width="0.1524" layer="91"/>
+</segment>
+</net>
+<net name="N$8" class="0">
+<segment>
+<pinref part="U$3" gate="G$1" pin="D5"/>
+<wire x1="162.56" y1="182.88" x2="162.56" y2="139.7" width="0.1524" layer="91"/>
+<wire x1="162.56" y1="139.7" x2="109.22" y2="139.7" width="0.1524" layer="91"/>
+<wire x1="109.22" y1="139.7" x2="109.22" y2="121.92" width="0.1524" layer="91"/>
+<wire x1="109.22" y1="121.92" x2="83.82" y2="121.92" width="0.1524" layer="91"/>
+<pinref part="U$1" gate="G$1" pin="ECHO"/>
+<wire x1="83.82" y1="121.92" x2="83.82" y2="134.62" width="0.1524" layer="91"/>
+</segment>
+</net>
+<net name="N$9" class="0">
+<segment>
+<pinref part="IC2" gate="G$1" pin="OUT"/>
+<wire x1="208.28" y1="187.96" x2="208.28" y2="111.76" width="0.1524" layer="91"/>
+<wire x1="208.28" y1="111.76" x2="165.1" y2="111.76" width="0.1524" layer="91"/>
+<pinref part="U$3" gate="G$1" pin="A0"/>
+<wire x1="165.1" y1="111.76" x2="165.1" y2="121.92" width="0.1524" layer="91"/>
+</segment>
+</net>
+<net name="N$10" class="0">
+<segment>
+<pinref part="U$2" gate="G$1" pin="AO"/>
+<pinref part="U$3" gate="G$1" pin="A1"/>
+<wire x1="193.04" y1="88.9" x2="167.64" y2="88.9" width="0.1524" layer="91"/>
+<wire x1="167.64" y1="88.9" x2="167.64" y2="121.92" width="0.1524" layer="91"/>
+</segment>
+</net>
+<net name="VSS" class="0">
+<segment>
+<pinref part="X1" gate="G$1" pin="VSS"/>
+<wire x1="60.96" y1="203.2" x2="60.96" y2="210.82" width="0.1524" layer="91"/>
+<wire x1="60.96" y1="210.82" x2="40.64" y2="210.82" width="0.1524" layer="91"/>
+<wire x1="40.64" y1="210.82" x2="40.64" y2="111.76" width="0.1524" layer="91"/>
+<pinref part="U$1" gate="G$1" pin="VCC"/>
+<wire x1="78.74" y1="134.62" x2="78.74" y2="111.76" width="0.1524" layer="91"/>
+<wire x1="78.74" y1="111.76" x2="78.74" y2="106.68" width="0.1524" layer="91"/>
+<wire x1="78.74" y1="106.68" x2="152.4" y2="106.68" width="0.1524" layer="91"/>
+<pinref part="U$3" gate="G$1" pin="5V"/>
+<wire x1="152.4" y1="106.68" x2="152.4" y2="114.3" width="0.1524" layer="91"/>
+<wire x1="152.4" y1="114.3" x2="152.4" y2="121.92" width="0.1524" layer="91"/>
+<wire x1="40.64" y1="111.76" x2="78.74" y2="111.76" width="0.1524" layer="91"/>
+<junction x="78.74" y="111.76"/>
+<pinref part="IC2" gate="G$1" pin="IN"/>
+<wire x1="193.04" y1="187.96" x2="193.04" y2="114.3" width="0.1524" layer="91"/>
+<wire x1="193.04" y1="114.3" x2="152.4" y2="114.3" width="0.1524" layer="91"/>
+<junction x="152.4" y="114.3"/>
+<pinref part="U$2" gate="G$1" pin="VCC"/>
+<wire x1="193.04" y1="96.52" x2="152.4" y2="96.52" width="0.1524" layer="91"/>
+<wire x1="152.4" y1="96.52" x2="152.4" y2="106.68" width="0.1524" layer="91"/>
+<junction x="152.4" y="106.68"/>
+</segment>
+</net>
+<net name="VDD" class="0">
+<segment>
+<pinref part="X1" gate="G$1" pin="VDD"/>
+<wire x1="63.5" y1="203.2" x2="63.5" y2="210.82" width="0.1524" layer="91"/>
+<pinref part="X1" gate="G$1" pin="RW"/>
+<wire x1="63.5" y1="210.82" x2="71.12" y2="210.82" width="0.1524" layer="91"/>
+<wire x1="71.12" y1="210.82" x2="71.12" y2="203.2" width="0.1524" layer="91"/>
+<wire x1="71.12" y1="210.82" x2="81.28" y2="210.82" width="0.1524" layer="91"/>
+<junction x="71.12" y="210.82"/>
+<wire x1="81.28" y1="210.82" x2="81.28" y2="205.74" width="0.1524" layer="91"/>
+<wire x1="81.28" y1="205.74" x2="96.52" y2="205.74" width="0.1524" layer="91"/>
+<pinref part="X1" gate="G$1" pin="A"/>
+<wire x1="96.52" y1="205.74" x2="96.52" y2="203.2" width="0.1524" layer="91"/>
+<wire x1="71.12" y1="210.82" x2="71.12" y2="167.64" width="0.1524" layer="91"/>
+<pinref part="IC2" gate="G$1" pin="GND"/>
+<wire x1="200.66" y1="180.34" x2="200.66" y2="116.84" width="0.1524" layer="91"/>
+<wire x1="200.66" y1="116.84" x2="157.48" y2="116.84" width="0.1524" layer="91"/>
+<pinref part="U$3" gate="G$1" pin="GND1"/>
+<wire x1="157.48" y1="116.84" x2="157.48" y2="121.92" width="0.1524" layer="91"/>
+<pinref part="U$1" gate="G$1" pin="GND"/>
+<wire x1="86.36" y1="134.62" x2="86.36" y2="116.84" width="0.1524" layer="91"/>
+<wire x1="86.36" y1="116.84" x2="157.48" y2="116.84" width="0.1524" layer="91"/>
+<junction x="157.48" y="116.84"/>
+<wire x1="71.12" y1="167.64" x2="157.48" y2="167.64" width="0.1524" layer="91"/>
+<wire x1="157.48" y1="167.64" x2="157.48" y2="121.92" width="0.1524" layer="91"/>
+<junction x="157.48" y="121.92"/>
+</segment>
+</net>
+<net name="N$11" class="0">
+<segment>
+<pinref part="U$2" gate="G$1" pin="GND"/>
+<pinref part="U$3" gate="G$1" pin="GND2"/>
+<wire x1="193.04" y1="93.98" x2="154.94" y2="93.98" width="0.1524" layer="91"/>
+<wire x1="154.94" y1="93.98" x2="154.94" y2="121.92" width="0.1524" layer="91"/>
+</segment>
+</net>
 </nets>
 </sheet>
